Commit message: Document keyboard teleop and improve robot model

File: models/robot.urdf.xacro (robot description, xacro)
@@ -73,4 +73,8 @@
                               h="${wheel_width}"/>
     </link>
+      <gazebo reference="${name}_wheel">
+        <mu1 value="0.9"/>
+        <mu2 value="0.9"/>
+      </gazebo>
     <joint name="${name}_wheel_joint" type="revolute">
       <parent link="base_link"/>
@@ -92,4 +96,22 @@
       </material>
     </visual>
+    <visual>
+      <origin xyz="0 0 0.04" rpy="0 0 0"/>
+      <geometry>
+        <box size="0.24 0.13 0.014"/>
+      </geometry>
+      <material name="dark_blue">
+        <color rgba="0.08 0.12 0.2 1"/>
+      </material>
+    </visual>
+    <visual>
+      <origin xyz="0.154 0 0" rpy="0 0 0"/>
+      <geometry>
+        <box size="0.016 0.17 0.04"/>
+      </geometry>
+      <material name="bumper">
+        <color rgba="0.07 0.08 0.09 1"/>
+      </material>
+    </visual>
     <collision>
       <origin xyz="0 0 0" rpy="0 0 0"/>
@@ -133,4 +155,8 @@
     <xacro:cylinder_inertia m="${wheel_mass}" r="${wheel_radius}" h="${wheel_width}"/>
   </link>
+  <gazebo reference="front_left_wheel_link">
+    <mu1 value="0.9"/>
+    <mu2 value="0.9"/>
+  </gazebo>
   <joint name="front_left_wheel_joint" type="revolute">
     <parent link="front_left_steer_link"/>
@@ -169,4 +195,8 @@
     <xacro:cylinder_inertia m="${wheel_mass}" r="${wheel_radius}" h="${wheel_width}"/>
   </link>
+  <gazebo reference="front_right_wheel_link">
+    <mu1 value="0.9"/>
+    <mu2 value="0.9"/>
+  </gazebo>
   <joint name="front_right_wheel_joint" type="revolute">
     <parent link="front_right_steer_link"/>
@@ -239,8 +269,8 @@
       <left_steering_joint>front_left_steer_joint</left_steering_joint>
       <right_steering_joint>front_right_steer_joint</right_steering_joint>
-      <kingpin_width>0.2</kingpin_width>
+      <kingpin_width>0.192</kingpin_width>
       <steering_limit>0.5</steering_limit>
-      <wheel_base>0.3</wheel_base>
-      <wheel_separation>0.2</wheel_separation>
+      <wheel_base>0.257</wheel_base>
+      <wheel_separation>0.192</wheel_separation>
       <wheel_radius>0.05</wheel_radius>
       <topic>/cmd_vel</topic>
